File: pimentero.kicad_sch (KiCad schematic)
At the start: 12 parts, among them J1 Conn_01x04_Female, Q1 MMBF5457

Commit message: v0.2: added volume pot (only pad for lug 1; lug 2 = GND, lug 3 = NC)
Parts:
- added J2: Volume A500k lug 1, Connector_PinHeader_2.54mm:PinHeader_1x01_P2.54mm_Vertical, symbol Connector:Conn_01x01_Female
Connections:
- net at C3.1, R3.1: now also Q1.1 (D); no longer Q1.2 (S)
- net at C4.2, R5.1, R6.1: now also J2.1 (Pin_1)
- net at C4.1, R4.2: now also Q1.2 (S); no longer Q1.1 (D)
Changed lines of the file:
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@@
+    (stroke (width 0) (type solid) (color 0 0 0 0))
+  )
+  (wire (pts (xy 95.885 33.655) (xy 95.885 43.815))
     (stroke (width 0) (type solid) (color 0 0 0 0))
   )
@@
     )
     (property "Datasheet" "" (id 3) (at 95.885 66.04 0)
+      (effects (font (size 1.27 1.27)) hide)
+    )
+  )
+  (symbol (lib_id "Connector:Conn_01x01_Female") (at 100.965 33.655 0) (unit 1)
+    (in_bom yes) (on_board yes)
+    (property "Reference" "J2" (id 0) (at 101.6763 32.9628 0)
+      (effects (font (size 1.27 1.27)) (justify left))
+    )
+    (property "Value" "Volume A500k lug 1" (id 1) (at 101.6763 35.2615 0)
+      (effects (font (size 1.27 1.27)) (justify left))
+    )
+    (property "Footprint" "Connector_PinHeader_2.54mm:PinHeader_1x01_P2.54mm_Vertical" (id 2) (at 100.965 33.655 0)
+      (effects (font (size 1.27 1.27)) hide)
+    )
+    (property "Datasheet" "~" (id 3) (at 100.965 33.655 0)
       (effects (font (size 1.27 1.27)) hide)
     )
@@
     )
   )
-  (symbol (lib_id "rockola_symbols:MMBFJ201") (at 72.39 49.53 0) (unit 1)
-    (in_bom yes) (on_board yes)
-    (property "Reference" "Q1" (id 0) (at 77.2415 48.3806 0)
-      (effects (font (size 1.27 1.27)) (justify left))
-    )
-    (property "Value" "MMBF5457" (id 1) (at 77.2415 50.6793 0)
-      (effects (font (size 1.27 1.27)) (justify left))
-    )
-    (property "Footprint" "Package_TO_SOT_SMD:SOT-23" (id 2) (at 77.47 51.435 0)
+  (symbol (lib_id "rockola_symbols:MMBFJ201") (at 72.39 49.53 0) (mirror x) (unit 1)
+    (in_bom yes) (on_board yes)
+    (property "Reference" "Q1" (id 0) (at 77.2415 50.6794 0)
+      (effects (font (size 1.27 1.27)) (justify left))
+    )
+    (property "Value" "MMBF5457" (id 1) (at 77.2415 48.3807 0)
+      (effects (font (size 1.27 1.27)) (justify left))
+    )
+    (property "Footprint" "Package_TO_SOT_SMD:SOT-23" (id 2) (at 77.47 47.625 0)
       (effects (font (size 1.27 1.27) italic) (justify left) hide)
     )
@@
       (reference "J1") (unit 1)
     )
+    (path "/b1dfd13b-250d-4271-b515-73cc2907d4f7"
+      (reference "J2") (unit 1)
+    )
     (path "/bca0b9b2-fc4c-4cae-95c0-90e6404b50df"
